File: pcb/pcb_files/hackpad_pcb.kicad_sch (KiCad schematic)
At the start: 1 part, among them U1 MOUDLE-SEEEDUINO-XIAO

Commit message: a
Changed lines of the file:
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@@
 	(symbol
 		(lib_id "XIAO_RP2040:MOUDLE-SEEEDUINO-XIAO")
-		(at 115.57 96.52 0)
+		(at 110.49 96.52 0)
 		(unit 1)
 		(body_style 1)
@@
 		(fields_autoplaced yes)
 		(property "Reference" "U1"
-			(at 116.84 81.28 0)
+			(at 111.76 81.28 0)
 			(show_name no)
 			(do_not_autoplace no)
@@
 		)
 		(property "Value" "MOUDLE-SEEEDUINO-XIAO"
-			(at 116.84 83.82 0)
+			(at 111.76 83.82 0)
 			(show_name no)
 			(do_not_autoplace no)
@@
 		)
 		(property "Footprint" ""
-			(at 99.06 93.98 0)
+			(at 93.98 93.98 0)
 			(hide yes)
 			(show_name no)
@@
 		)
 		(property "Datasheet" ""
-			(at 99.06 93.98 0)
+			(at 93.98 93.98 0)
 			(hide yes)
 			(show_name no)
@@
 		)
 		(property "Description" ""
-			(at 115.57 96.52 0)
+			(at 110.49 96.52 0)
 			(hide yes)
 			(show_name no)
@@
 			)
 		)
+		(pin "9"
+		)
+		(pin "3"
+		)
+		(pin "5"
+		)
+		(pin "7"
+		)
 		(pin "1"
 		)
-		(pin "6"
+		(pin "14"
 		)
 		(pin "10"
@@
 		(pin "11"
 		)
-		(pin "3"
+		(pin "6"
+		)
+		(pin "13"
 		)
 		(pin "8"
@@
 		(pin "2"
 		)
-		(pin "5"
-		)
-		(pin "7"
-		)
-		(pin "9"
-		)
 		(pin "12"
 		)
-		(pin "14"
-		)
-		(pin "13"
-		)
 		(instances

Commit message: b
Parts:
- added D1: 1N4148, Diode_THT:D_DO-35_SOD27_P7.62mm_Horizontal, symbol Diode:1N4148
- added SW1, SW2, SW3, SW4, SW5, SW6: SW_Push, symbol Switch:SW_Push

Commit message: Modified Schematic
Parts:
- added D2, D3, D4, D5, D6: 1N4148, Diode_THT:D_DO-35_SOD27_P7.62mm_Horizontal, symbol Diode:1N4148
- added SW7: RotaryEncoder_Switch, symbol Device:RotaryEncoder_Switch
- added U2: ER_OLEDM0.91_1x-I2C, Display:ER_OLEDM0.91_1x-I2C, symbol Display_Graphic:ER_OLEDM0.91_1x-I2C
Connections:
- net Row 1: now also U1.2 (PA4_A1_D1), D4.1 (K), D5.1 (K), D6.1 (K)
- net at SW1.1: now also D1.2 (A)
- net Col 0: now reaches SW1.2
- net Col 0: now also D1.1 (K), SW2.2, SW4.2, SW5.2, U1.1 (PA02_A0_D0), U1.10 (PA5_A9_D9_MISO), U1.9 (PA7_A8_D8_SCK), D2.1 (K), D3.1 (K)
- net at SW3.1: now also D3.2 (A)
- net GND: now reaches SW3.2
- net GND: now also SW6.2, U1.13 (GND), U1.8 (PB09_A7_D7_RX), SW7.C, U2.1 (GND)
- net at SW5.1: now also D5.2 (A)
- net at U1.12 (3V3): no longer names the net of U1.12 (3V3)
- net at U1.12 (3V3): now also U2.2 (VCC)
- net SCL: now reaches U1.3 (PA10_A2_D2)
- net SCL: now also U2.3 (SCL)
- net LDA: now reaches U1.4 (PA11_A3_D3)
- net LDA: now also U2.4 (SDA)
- net A: now reaches U1.5 (PA8_A4_D4_SDA)
- net A: now also SW7.A
- net B: now reaches U1.6 (PA9_A5_D5_SCL)
- net B: now also SW7.B
- net at SW4.1: now also D4.2 (A)
- net at SW6.1: now also D6.2 (A)
- net at SW2.1: now also D2.2 (A)
- no-connect marks 0 -> 5
Other:
- moved on the sheet: D1, SW1

Commit message: Finished the schematic
Parts:
- SW1, SW2, SW3, SW4, SW5, SW6: footprint (none) -> Button_Switch_Keyboard:SW_Cherry_MX_1.00u_PCB
- SW7: footprint (none) -> Rotary_Encoder:RotaryEncoder_Alps_EC11E-Switch_Vertical_H20mm
- U1: footprint (none) -> footprint:XIAO-Generic-Hybrid-14P-2.54-21X17.8MM
Connections:
- net GND: no longer SW3.2, SW6.2, U1.8 (PB09_A7_D7_RX)
- net 3V3: now reaches U1.12 (3V3), U2.2 (VCC)
- net Col 0 renamed Col_1
- net Col_1: now also U1.8 (PB09_A7_D7_RX); no longer U1.10 (PA5_A9_D9_MISO)
- net LDA renamed SDA
- net Row 1 renamed Row_1
- new net Col_0: SW3.2, SW6.2, U1.10 (PA5_A9_D9_MISO)
Other:
- note added: "OLED DISPLAY"
- note added: "ROTARY ENCODER"
- note added: "SWITCH MATRIX"
- moved on the sheet: D1, D2, D3, D4, D5, D6, SW1, SW2, SW3, SW4, SW5, SW6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

Commit message: Updated the PCB
Parts:
- removed D3: 1N4148, Diode_THT:D_DO-35_SOD27_P7.62mm_Horizontal, symbol Diode:1N4148
- removed SW3: SW_Push, Button_Switch_Keyboard:SW_Cherry_MX_1.00u_PCB, symbol Switch:SW_Push
Connections:
- net Col_1: no longer SW1.2, SW4.2, U1.8 (PB09_A7_D7_RX)
- new net Col_2: SW1.2, SW4.2, U1.8 (PB09_A7_D7_RX)
